Commit message: Update arm.ros2_control.xacro

File: description/ros2_control/arm.ros2_control.xacro (robot description, xacro)
@@ -28,5 +28,5 @@
         <state_interface name="position" />
       </joint>
-      <joint name="joint3">
+      <joint name="joint2">
         <command_interface name="position">
           <param name="min">-1</param>
@@ -35,5 +35,5 @@
         <state_interface name="position" />
       </joint>
-      <joint name="joint4">
+      <joint name="joint3">
         <command_interface name="position">
           <param name="min">-1</param>
