Commit message: Update arm_description.urdf.xacro

File: description/rrbot/urdf/arm_description.urdf.xacro (robot description, xacro)
@@ -5,5 +5,5 @@
       <limit lower="-3.14000" upper="3.14000" effort="0.00000" velocity="0.00000" />
       <origin rpy="-3.14159 -0.00000 1.57062" xyz="0.00089 -0.00025 0.00205" />
-      <parent link="root.000" />
+      <parent link="link0" />
       <child link="link1" />
       <axis xyz="0.00000 0.00000 -1.00000" />
@@ -16,5 +16,5 @@
       <axis xyz="0.00000 0.00000 -1.00000" />
     </joint>
-    <joint name="joint3" type="revolute">
+    <joint name="joint2" type="revolute">
       <limit lower="-3.14000" upper="3.14000" effort="0.00000" velocity="0.00000" />
       <origin rpy="0.00000 0.00000 0.00000" xyz="-0.09876 0.00001 -0.00008" />
@@ -23,5 +23,5 @@
       <axis xyz="0.00000 0.00000 -1.00000" />
     </joint>
-    <joint name="joint4" type="revolute">
+    <joint name="joint3" type="revolute">
       <limit lower="-3.14000" upper="3.14000" effort="0.00000" velocity="0.00000" />
       <origin rpy="-0.00000 -0.00000 -0.00000" xyz="-0.09983 0.00001 -0.00027" />
@@ -37,4 +37,10 @@
         <mass value="0.20000" />
       </inertial>
+      <visual name="link_1">
+      <origin rpy="-0.00000 -0.00000 -0.00000" xyz="-0.00000 0.00000 -0.00000"/>
+      <geometry>
+         <mesh filename="file://$(find ros2_control_demo_example_9)/meshes/stl/Cube.019.stl" scale="1.00000 1.00000 1.00000" />
+      </geometry>
+    </visual>
     </link>
     <link name="link2">
@@ -67,7 +73,7 @@
     <link name="link4">
       <inertial>
-        <inertia ixx="0.00100" ixy="0.00000" ixz="0.00000" iyy="0.00100" iyz="0.00000" izz="0.00100" />
-        <origin rpy="0.00000 0.00000 0.00000" xyz="-0.00000 -0.00000 0.00000" />
-        <mass value="0.20000" />
+        <inertia ixx="0.00131" ixy="0.00000" ixz="0.00000" iyy="0.00131" iyz="0.00000" izz="0.00131"/>
+        <origin rpy="0.00000 0.00000 0.00000" xyz="0.00084 -0.00000 0.00027"/>
+        <mass value="0.20000"/>
       </inertial>
       <visual name="link_4">
@@ -78,6 +84,6 @@
       </visual>
     </link>
-    <link name="root.000">
-      <visual name="base">
+    <link name="link0">
+      <visual name="link_0">
         <origin rpy="0.00000 0.00000 -0.00000" xyz="-0.00000 0.00000 0.00000" />
         <geometry>
@@ -89,5 +95,5 @@
       <origin xyz="0 0 0" rpy="0 0 0" />
       <parent link="${parent}" />
-      <child link="root.000" />
+      <child link="link0" />
     </joint>
     </xacro:macro>

Commit message: Update arm_description.urdf.xacro

File: description/rrbot/urdf/arm_description.urdf.xacro (robot description, xacro)
@@ -85,4 +85,9 @@
     </link>
     <link name="link0">
+      <inertial>
+        <inertia ixx="0.00207" ixy="0.00000" ixz="0.00000" iyy="0.00207" iyz="0.00000" izz="0.00207"/>
+        <origin rpy="0.00000 0.00000 0.00000" xyz="0.00000 -0.00000 0.00000"/>
+        <mass value="0.30000"/>
+      </inertial>
       <visual name="link_0">
         <origin rpy="0.00000 0.00000 -0.00000" xyz="-0.00000 0.00000 0.00000" />

Commit message: Update arm_description.urdf.xacro

File: description/rrbot/urdf/arm_description.urdf.xacro (robot description, xacro)
@@ -37,5 +37,5 @@
         <mass value="0.20000" />
       </inertial>
-      <visual name="link_1">
+      <visual>
       <origin rpy="-0.00000 -0.00000 -0.00000" xyz="-0.00000 0.00000 -0.00000"/>
       <geometry>
@@ -51,5 +51,5 @@
         <mass value="0.20000" />
       </inertial>
-      <visual name="link_2">
+      <visual>
         <origin rpy="-0.00002 -0.00000 0.00000" xyz="-0.00000 0.00000 -0.00000" />
         <geometry>
@@ -64,5 +64,5 @@
         <mass value="0.20000" />
       </inertial>
-      <visual name="link_3">
+      <visual>
         <origin rpy="-0.00002 -0.00000 0.00000" xyz="-0.00000 -0.00000 -0.00000" />
         <geometry>
@@ -77,5 +77,5 @@
         <mass value="0.20000"/>
       </inertial>
-      <visual name="link_4">
+      <visual>
         <origin rpy="-0.00002 -0.00000 0.00000" xyz="-0.00000 0.00000 0.00000" />
         <geometry>
@@ -90,5 +90,5 @@
         <mass value="0.30000"/>
       </inertial>
-      <visual name="link_0">
+      <visual>
         <origin rpy="0.00000 0.00000 -0.00000" xyz="-0.00000 0.00000 0.00000" />
         <geometry>
