Commit message: changing namespace name

File: description/gazebo/rrbot.gazebo.xacro (robot description, xacro)
@@ -9,5 +9,5 @@
     <gazebo>
       <plugin filename="gz_ros2_control-system" name="gz_ros2_control::GazeboSimROS2ControlPlugin">
-        <parameters>$(find ros2_control_demo_example_9)/config/rrbot_controllers.yaml</parameters>
+        <parameters>$(find simple_arm)/config/rrbot_controllers.yaml</parameters>
       </plugin>
     </gazebo>

File: description/ros2_control/arm.ros2_control.xacro (robot description, xacro)
@@ -8,6 +8,6 @@
         </xacro:if>
         <xacro:unless value="${use_gazebo}">
-          <plugin>ros2_control_demo_example_9/RRBotSystemPositionOnlyHardware</plugin>
-          <param name="example_param_hw_start_duration_sec">5</param>
+          <plugin>simple_arm/RRBotSystemPositionOnlyHardware</plugin>
+          <param name="example_param_hw_start_duration_sec">3</param>
           <param name="example_param_hw_stop_duration_sec">3.0</param>
           <param name="example_param_hw_slowdown">100</param>

File: description/rrbot/urdf/arm_description.urdf.xacro (robot description, xacro)
@@ -40,5 +40,5 @@
       <origin rpy="-0.00000 -0.00000 -0.00000" xyz="-0.00000 0.00000 -0.00000"/>
       <geometry>
-         <mesh filename="file://$(find ros2_control_demo_example_9)/meshes/stl/Cube.019.stl" scale="1.00000 1.00000 1.00000" />
+         <mesh filename="file://$(find simple_arm)/meshes/stl/Cube.019.stl" scale="1.00000 1.00000 1.00000" />
       </geometry>
     </visual>
@@ -54,5 +54,5 @@
         <origin rpy="-0.00002 -0.00000 0.00000" xyz="-0.00000 0.00000 -0.00000" />
         <geometry>
-          <mesh filename="file://$(find ros2_control_demo_example_9)/meshes/stl/Cube.010.stl" scale="1.00000 1.00000 1.00000" />
+          <mesh filename="file://$(find simple_arm)/meshes/stl/Cube.010.stl" scale="1.00000 1.00000 1.00000" />
         </geometry>
       </visual>
@@ -67,5 +67,5 @@
         <origin rpy="-0.00002 -0.00000 0.00000" xyz="-0.00000 -0.00000 -0.00000" />
         <geometry>
-          <mesh filename="file://$(find ros2_control_demo_example_9)/meshes/stl/Cube.013.stl" scale="1.00000 1.00000 1.00000" />
+          <mesh filename="file://$(find simple_arm)/meshes/stl/Cube.013.stl" scale="1.00000 1.00000 1.00000" />
         </geometry>
       </visual>
@@ -80,5 +80,5 @@
         <origin rpy="-0.00002 -0.00000 0.00000" xyz="-0.00000 0.00000 0.00000" />
         <geometry>
-          <mesh filename="file://$(find ros2_control_demo_example_9)/meshes/stl/Cube.014.stl" scale="1.00000 1.00000 1.00000" />
+          <mesh filename="file://$(find simple_arm)/meshes/stl/Cube.014.stl" scale="1.00000 1.00000 1.00000" />
         </geometry>
       </visual>
@@ -93,5 +93,5 @@
         <origin rpy="0.00000 0.00000 -0.00000" xyz="-0.00000 0.00000 0.00000" />
         <geometry>
-          <mesh filename="file://$(find ros2_control_demo_example_9)/meshes/stl/Cube.018.stl" scale="1.00000 1.00000 1.00000" />
+          <mesh filename="file://$(find simple_arm)/meshes/stl/Cube.018.stl" scale="1.00000 1.00000 1.00000" />
         </geometry>
       </visual>

File: description/urdf/arm.urdf.xacro (robot description, xacro)
@@ -10,11 +10,11 @@
     <!-- Import RRBot macro -->
     <xacro:include
-        filename="$(find ros2_control_demo_example_9)/rrbot/urdf/arm_description.urdf.xacro" />
+        filename="$(find simple_arm)/rrbot/urdf/arm_description.urdf.xacro" />
     <!-- Import Rviz colors -->
     <xacro:include
-        filename="$(find ros2_control_demo_example_9)/rrbot/urdf/arm.materials.xacro" />
+        filename="$(find simple_arm)/rrbot/urdf/arm.materials.xacro" />
     <!-- Import RRBot ros2_control description -->
     <xacro:include
-        filename="$(find ros2_control_demo_example_9)/ros2_control/arm.ros2_control.xacro" />
+        filename="$(find simple_arm)/ros2_control/arm.ros2_control.xacro" />
     <!-- Used for fixing robot -->
     <link name="world" />
@@ -26,5 +26,5 @@
     <xacro:if value="$(arg use_gazebo)">
         <!-- Import Gazebo Classic definitions + plugin -->
-        <xacro:include filename="$(find ros2_control_demo_example_9)/gazebo/rrbot.gazebo.xacro" />
+        <xacro:include filename="$(find simple_arm)/gazebo/rrbot.gazebo.xacro" />
         <xacro:rrbot_gazebo prefix="$(arg prefix)" />
     </xacro:if>
